Commit message: Testing pointcloud filtering components.

File: pacifica_sensor_kit_description/urdf/sensor_kit.xacro (robot description, xacro)
@@ -21,12 +21,12 @@
     <xacro:property name="calibration" value="${xacro.load_yaml('$(arg config_dir)/sensor_kit_calibration.yaml')}"/>
     <!-- lidar -->
-    <xacro:VLS-128 parent="sensor_kit_base_link" name="velodyne_top" topic="/points_raw" hz="10" samples="220" gpu="$(arg gpu)">
+    <xacro:VLS-128 parent="sensor_kit_base_link" name="quanergy" topic="/quanergy/points_raw" hz="15" samples="220" gpu="$(arg gpu)">
       <origin
-        xyz="${calibration['sensor_kit_base_link']['velodyne_top_base_link']['x']}
-             ${calibration['sensor_kit_base_link']['velodyne_top_base_link']['y']}
-             ${calibration['sensor_kit_base_link']['velodyne_top_base_link']['z']}"
-        rpy="${calibration['sensor_kit_base_link']['velodyne_top_base_link']['roll']}
-             ${calibration['sensor_kit_base_link']['velodyne_top_base_link']['pitch']}
-             ${calibration['sensor_kit_base_link']['velodyne_top_base_link']['yaw']}"
+        xyz="${calibration['sensor_kit_base_link']['quanergy_link']['x']}
+             ${calibration['sensor_kit_base_link']['quanergy_link']['y']}
+             ${calibration['sensor_kit_base_link']['quanergy_link']['z']}"
+        rpy="${calibration['sensor_kit_base_link']['quanergy_link']['roll']}
+             ${calibration['sensor_kit_base_link']['quanergy_link']['pitch']}
+             ${calibration['sensor_kit_base_link']['quanergy_link']['yaw']}"
       />
     </xacro:VLS-128>
@@ -112,26 +112,26 @@
     <!-- gnss -->
     <xacro:imu_macro
-      name="gnss"
+      name="yahboo_gnss"
       parent="sensor_kit_base_link"
       namespace=""
-      x="${calibration['sensor_kit_base_link']['gnss_link']['x']}"
-      y="${calibration['sensor_kit_base_link']['gnss_link']['y']}"
-      z="${calibration['sensor_kit_base_link']['gnss_link']['z']}"
-      roll="${calibration['sensor_kit_base_link']['gnss_link']['roll']}"
-      pitch="${calibration['sensor_kit_base_link']['gnss_link']['pitch']}"
-      yaw="${calibration['sensor_kit_base_link']['gnss_link']['yaw']}"
-      fps="100"
+      x="${calibration['sensor_kit_base_link']['yahboom/gnss_link']['x']}"
+      y="${calibration['sensor_kit_base_link']['yahboom/gnss_link']['y']}"
+      z="${calibration['sensor_kit_base_link']['yahboom/gnss_link']['z']}"
+      roll="${calibration['sensor_kit_base_link']['yahboom/gnss_link']['roll']}"
+      pitch="${calibration['sensor_kit_base_link']['yahboom/gnss_link']['pitch']}"
+      yaw="${calibration['sensor_kit_base_link']['yahboom/gnss_link']['yaw']}"
+      fps="10"
     />
     <xacro:imu_macro
-      name="gnss"
+      name="aceinna_gnss"
       parent="sensor_kit_base_link"
       namespace=""
-      x="${calibration['sensor_kit_base_link']['gnss_link']['x']}"
-      y="${calibration['sensor_kit_base_link']['gnss_link']['y']}"
-      z="${calibration['sensor_kit_base_link']['gnss_link']['z']}"
-      roll="${calibration['sensor_kit_base_link']['gnss_link']['roll']}"
-      pitch="${calibration['sensor_kit_base_link']['gnss_link']['pitch']}"
-      yaw="${calibration['sensor_kit_base_link']['gnss_link']['yaw']}"
-      fps="100"
+      x="${calibration['sensor_kit_base_link']['aceinna/gnss_link']['x']}"
+      y="${calibration['sensor_kit_base_link']['aceinna/gnss_link']['y']}"
+      z="${calibration['sensor_kit_base_link']['aceinna/gnss_link']['z']}"
+      roll="${calibration['sensor_kit_base_link']['aceinna/gnss_link']['roll']}"
+      pitch="${calibration['sensor_kit_base_link']['aceinna/gnss_link']['pitch']}"
+      yaw="${calibration['sensor_kit_base_link']['aceinna/gnss_link']['yaw']}"
+      fps="10"
     />
   </xacro:macro>

File: pacifica_sensor_kit_description/urdf/sensors.xacro (robot description, xacro)
@@ -17,15 +17,15 @@
     yaw="${calibration['base_link']['sensor_kit_base_link']['yaw']}"
   />
-  <!-- embedded sensors -->
-  <xacro:include filename="$(find velodyne_description)/urdf/VLP-16.urdf.xacro"/>
-  <xacro:VLP-16 parent="base_link" name="velodyne_rear" topic="velodyne_rear/velodyne_points" hz="10" samples="220" gpu="false">
-    <origin
-      xyz="${calibration['base_link']['velodyne_rear_base_link']['x']}
-           ${calibration['base_link']['velodyne_rear_base_link']['y']}
-           ${calibration['base_link']['velodyne_rear_base_link']['z']}"
-      rpy="${calibration['base_link']['velodyne_rear_base_link']['roll']}
-           ${calibration['base_link']['velodyne_rear_base_link']['pitch']}
-           ${calibration['base_link']['velodyne_rear_base_link']['yaw']}"
-    />
-  </xacro:VLP-16>
+  <!-- embedded sensors. Todo: add aceinna IMU_link and optionally yahboom imu_link -->
+<!--  <xacro:include filename="$(find velodyne_description)/urdf/VLP-16.urdf.xacro"/>-->
+<!--  <xacro:VLP-16 parent="base_link" name="velodyne_rear" topic="velodyne_rear/velodyne_points" hz="10" samples="220" gpu="false">-->
+<!--    <origin-->
+<!--      xyz="${calibration['base_link']['velodyne_rear_base_link']['x']}-->
+<!--           ${calibration['base_link']['velodyne_rear_base_link']['y']}-->
+<!--           ${calibration['base_link']['velodyne_rear_base_link']['z']}"-->
+<!--      rpy="${calibration['base_link']['velodyne_rear_base_link']['roll']}-->
+<!--           ${calibration['base_link']['velodyne_rear_base_link']['pitch']}-->
+<!--           ${calibration['base_link']['velodyne_rear_base_link']['yaw']}"-->
+<!--    />-->
+<!--  </xacro:VLP-16>-->
 </robot>

Commit message: Testing pointcloud filtering components.

File: pacifica_sensor_kit_description/urdf/sensor_kit.xacro (robot description, xacro)
@@ -21,17 +21,6 @@
     <xacro:property name="calibration" value="${xacro.load_yaml('$(arg config_dir)/sensor_kit_calibration.yaml')}"/>
     <!-- lidar -->
-    <xacro:VLS-128 parent="sensor_kit_base_link" name="quanergy" topic="/quanergy/points_raw" hz="15" samples="220" gpu="$(arg gpu)">
-      <origin
-        xyz="${calibration['sensor_kit_base_link']['quanergy_link']['x']}
-             ${calibration['sensor_kit_base_link']['quanergy_link']['y']}
-             ${calibration['sensor_kit_base_link']['quanergy_link']['z']}"
-        rpy="${calibration['sensor_kit_base_link']['quanergy_link']['roll']}
-             ${calibration['sensor_kit_base_link']['quanergy_link']['pitch']}
-             ${calibration['sensor_kit_base_link']['quanergy_link']['yaw']}"
-      />
-    </xacro:VLS-128>
-    <!-- depth camera. todo test azure urdf -->
-    <xacro:macro name="azure_kinect_macro" params="parent x y z roll pitch yaw">
-      <joint name="azure_kinect/camera_link" type="fixed">
+    <xacro:macro name="quanergy_lidar_macro" params="parent x y z roll pitch yaw">
+      <joint name="quanergy_base_joint" type="fixed">
         <origin
           xyz="${x}
@@ -43,10 +32,59 @@
         />
         <parent link="${parent}"/>
-        <child link="camera_base"/>
+        <child link="quanergy_base_link"/>
       </joint>
-      <xacro:azure-kinect>
-<!--          <xacro:insert_block name="origin" />-->
-      </xacro:azure-kinect>
+      <link name="quanergy_base_link">
+<!--        <origin rpy="0 0 0" xyz="0 0 0"/>-->
+      </link>
+      <joint name="quanergy_link" type="fixed">
+        <origin xyz="0 0 0.2" rpy="0 0 0"/>
+        <parent link="quanergy_base_link"/>
+        <child link="quanergy_link" />
+      </joint>
+      <link name="quanergy_link">
+<!--        <origin rpy="0 0 0" xyz="0 0 0"/>-->
+      </link>
     </xacro:macro>
+    <xacro:quanergy_lidar_macro
+            parent="sensor_kit_base_link"
+            x="${calibration['sensor_kit_base_link']['quanergy_base_link']['x']}"
+            y="${calibration['sensor_kit_base_link']['quanergy_base_link']['y']}"
+            z="${calibration['sensor_kit_base_link']['quanergy_base_link']['z']}"
+            roll="${calibration['sensor_kit_base_link']['quanergy_base_link']['roll']}"
+            pitch="${calibration['sensor_kit_base_link']['quanergy_base_link']['pitch']}"
+            yaw="${calibration['sensor_kit_base_link']['quanergy_base_link']['yaw']}"
+    />
+    <!-- depth camera. -->
+    <xacro:macro name="azure_kinect_macro" params="parent x y z roll pitch yaw">
+      <joint name="azure_kinect_joint" type="fixed">
+        <origin
+          xyz="${x}
+               ${y}
+               ${z}"
+          rpy="${roll}
+               ${pitch}
+               ${yaw}"
+        />
+        <parent link="${parent}"/>
+        <child link="azure_kinect/camera_link"/>
+      </joint>
+      <link name="azure_kinect/camera_link">
+        <origin rpy="0 0 0" xyz="0 0 0"/>
+      </link>
+      <joint name="azure_base_joint" type="fixed">
+        <origin xyz="0 0 0" rpy="0 0 0"/>
+        <parent link="azure_kinect/camera_link"/>
+        <child link="camera_base" />
+      </joint>
+    </xacro:macro>
+    <xacro:azure_kinect_macro
+            parent="sensor_kit_base_link"
+            x="${calibration['sensor_kit_base_link']['azure_kinect/camera_link']['x']}"
+            y="${calibration['sensor_kit_base_link']['azure_kinect/camera_link']['y']}"
+            z="${calibration['sensor_kit_base_link']['azure_kinect/camera_link']['z']}"
+            roll="${calibration['sensor_kit_base_link']['azure_kinect/camera_link']['roll']}"
+            pitch="${calibration['sensor_kit_base_link']['azure_kinect/camera_link']['pitch']}"
+            yaw="${calibration['sensor_kit_base_link']['azure_kinect/camera_link']['yaw']}"
+    />
     <!-- monocular cameras -->
     <xacro:monocular_camera_macro

File: pacifica_sensor_kit_description/urdf/sensors.xacro (robot description, xacro)
@@ -12,5 +12,5 @@
     x="${calibration['base_link']['sensor_kit_base_link']['x']}"
     y="${calibration['base_link']['sensor_kit_base_link']['y']}"
-    z="${calibration['base_link']['sensor_kit_base_link']['z']} + vehicle_info['/**']['ros__parameters']['wheel_radius']}"
+    z="${calibration['base_link']['sensor_kit_base_link']['z'] + vehicle_info['/**']['ros__parameters']['wheel_radius']}"
     roll="${calibration['base_link']['sensor_kit_base_link']['roll']}"
     pitch="${calibration['base_link']['sensor_kit_base_link']['pitch']}"

Commit message: Modified GPS and IMU extrinsics.

File: pacifica_sensor_kit_description/urdf/sensor_kit.xacro (robot description, xacro)
@@ -148,4 +148,17 @@
       fov="1.3"
     />
+    <!-- IMUs -->
+    <xacro:imu_macro
+      name="yahboo_imu"
+      parent="sensor_kit_base_link"
+      namespace=""
+      x="${calibration['sensor_kit_base_link']['yahboom/imu_link']['x']}"
+      y="${calibration['sensor_kit_base_link']['yahboom/imu_link']['y']}"
+      z="${calibration['sensor_kit_base_link']['yahboom/imu_link']['z']}"
+      roll="${calibration['sensor_kit_base_link']['yahboom/imu_link']['roll']}"
+      pitch="${calibration['sensor_kit_base_link']['yahboom/imu_link']['pitch']}"
+      yaw="${calibration['sensor_kit_base_link']['yahboom/imu_link']['yaw']}"
+      fps="10"
+    />
     <!-- gnss -->
     <xacro:imu_macro

File: pacifica_sensor_kit_description/urdf/sensors.xacro (robot description, xacro)
@@ -17,4 +17,33 @@
     yaw="${calibration['base_link']['sensor_kit_base_link']['yaw']}"
   />
+  <!-- Rear axle -->
+  <xacro:macro name="static_tf_macro" params="parent child name x y z roll pitch yaw">
+    <joint name="${name}_joint" type="fixed">
+      <origin
+        xyz="${x}
+             ${y}
+             ${z}"
+        rpy="${roll}
+             ${pitch}
+             ${yaw}"
+      />
+      <parent link="${parent}"/>
+      <child link="${child}"/>
+    </joint>
+    <link name="${name}">
+      <origin rpy="0 0 0" xyz="0 0 0"/>
+    </link>
+  </xacro:macro>
+    <xacro:static_tf_macro
+      parent="base_link"
+      child="rear_axle_link"
+      name="rear_axle_joint"
+      x="${calibration['base_link']['rear_axle_link']['x']}"
+      y="${calibration['base_link']['rear_axle_link']['y']}"
+      z="${calibration['base_link']['rear_axle_link']['z']}"
+      roll="${calibration['base_link']['rear_axle_link']['roll']}"
+      pitch="${calibration['base_link']['rear_axle_link']['pitch']}"
+      yaw="${calibration['base_link']['rear_axle_link']['yaw']}"
+    />
   <!-- embedded sensors. Todo add aceinna IMU_link and optionally yahboom imu_link -->
 <!--  <xacro:include filename="$(find velodyne_description)/urdf/VLP-16.urdf.xacro"/>-->
